File: PCB/caelum_v2/caelum_v2.kicad_sch (KiCad schematic)
At the start: 29 parts, among them J1 Conn_01x06_Pin, J10 Conn_01x04_Pin, J3 Pulse1, J4 Batt, J6 Pulse2, J7 Conn_01x04_Pin, J8 DS18B20, Q1 FS8205A-FC, U1 DW01A, U2 MCP1825S, U3 ESP32-H2-SUPERMINI

Commit message: Update PCB V2
Parts:
- removed J1: Conn_01x06_Pin, Connector_JST:JST_SH_BM06B-SRSS-TB_1x06-1MP_P1.00mm_Vertical, symbol Connector:Conn_01x06_Pin
- removed J10: Conn_01x04_Pin, Connector_PinHeader_2.54mm:PinHeader_1x04_P2.54mm_Vertical, symbol Connector:Conn_01x04_Pin
- removed J6: Pulse2, Connector_PinHeader_2.54mm:PinHeader_1x02_P2.54mm_Vertical, symbol Connector:Conn_01x02_Pin
- added C10, C12, C13: 0.1µF, Capacitor_SMD:C_0805_2012Metric, symbol Device:C
- added C11: 1µF, Capacitor_SMD:C_0805_2012Metric, symbol Device:C
- added J1: SS445P, Connector_Hirose:Hirose_DF13C_CL535-0403-5-51_1x03-1MP_P1.25mm_Vertical, symbol Connector:Conn_01x03_Pin
- added J2: i2C Bus2, Connector_JST:JST_PH_B4B-PH-SM4-TB_1x04-1MP_P2.00mm_Vertical, symbol Connector:Conn_01x04_Pin
- added R6, R7: 4.7K, Resistor_SMD:R_0805_2012Metric, symbol Device:R
- added R8: 10K, Resistor_SMD:R_0805_2012Metric, symbol Device:R
- added U4: ~, Package_LGA:Bosch_LGA-8_2x2.5mm_P0.65mm_ClockwisePinNumbering, symbol caelum:DPS310
- C2, C4: value 1µF -> 10µF; footprint Capacitor_SMD:C_1206_3216Metric -> Capacitor_SMD:C_0805_2012Metric
- C6: footprint Capacitor_SMD:C_1206_3216Metric -> Capacitor_SMD:C_0805_2012Metric
- J3: footprint Connector_PinHeader_2.54mm:PinHeader_1x02_P2.54mm_Vertical -> Connector_Hirose:Hirose_DF13C_CL535-0402-2-51_1x02-1MP_P1.25mm_Vertical
- J7: value Conn_01x04_Pin -> I2C BUS1; footprint Connector_PinHeader_2.54mm:PinHeader_1x04_P2.54mm_Vertical -> Connector_JST:JST_PH_S4B-PH-SM4-TB_1x04-1MP_P2.00mm_Horizontal
- J8: footprint Connector_Molex:Molex_KK-254_AE-6410-03A_1x03_P2.54mm_Vertical -> Connector_Hirose:Hirose_DF13C_CL535-0403-5-51_1x03-1MP_P1.25mm_Vertical
Connections:
- net +3V3: now also J7.3 (Pin_3), C10.2, C11.2, C12.1, C13.1, J1.1 (Pin_1), J2.4 (Pin_4), R6.2, R7.2, R8.1, U4.2 (CSB), U4.5 (SDO), U4.6 (VDDIO), U4.8 (VDD); no longer J7.1 (Pin_1)
- net GPIO4: now also C9.1, R4.1, R5.2
- net OUT-: now also J7.4 (Pin_4), C10.1, C11.1, C12.2, C13.2, J1.3 (Pin_3), J2.3 (Pin_3), U4.1 (GND), U4.7 (GND); no longer J7.3 (Pin_3)
- net SCL: now also J7.2 (Pin_2), R7.1, U4.4 (SCK); no longer J7.4 (Pin_4)
- net SDA: now also J7.1 (Pin_1), R6.1, U4.3 (SDI); no longer J7.2 (Pin_2)
- net GPIO14: now reaches U3.6 (IO14)
- net GPIO14: now also J1.2 (Pin_2), R8.2
- net GPIO1 renamed SDA_2
- net SDA_2: now also J2.2 (Pin_2)
- net GPIO13: no longer names the net of U3.5 (IO13)
- net GPIO2 renamed SCL_2
- net SCL_2: now also J2.1 (Pin_1)
- net GPIO3: no longer names the net of U3.14 (IO3)
- removed net GPIO5: C9.1, R4.1, R5.2, U3.12 (IO5)
- no-connect marks 12 -> 14
Other:
- note added: "Anemometer"
- moved on the sheet: J7
