File: PCB/caelum_v2/caelum_v2.kicad_pcb (KiCad board)
At the start: 2 copper layers, 54 x 39.5 mm, 29 parts, among them J1 Conn_01x06_Pin, J10 Conn_01x04_Pin, J3 Pulse1, J4 Batt, J6 Pulse2, J7 Conn_01x04_Pin, J8 DS18B20, Q1 FS8205A-FC, U1 DW01A, U2 MCP1825S, U3 ESP32-H2-SUPERMINI

Commit message: Update PCB V2
Parts:
- removed J10: Conn_01x04_Pin, Connector_PinHeader_2.54mm:PinHeader_1x04_P2.54mm_Vertical
- removed J6: Pulse2, Connector_PinHeader_2.54mm:PinHeader_1x02_P2.54mm_Vertical
- added C10: 0.1µF, Capacitor_SMD:C_0805_2012Metric, F.Cu at (72.2, 29.0)
- added C11: 1µF, Capacitor_SMD:C_0805_2012Metric, F.Cu at (67.8, 29.6)
- added C12: 0.1µF, Capacitor_SMD:C_0805_2012Metric, F.Cu at (69.8, 34.0)
- added C13: 0.1µF, Capacitor_SMD:C_0805_2012Metric, F.Cu at (106.3, 48.0)
- added J2: i2C Bus2, Connector_JST:JST_PH_B4B-PH-SM4-TB_1x04-1MP_P2.00mm_Vertical, F.Cu at (109.8, 40.9)
- added R6: 4.7K, Resistor_SMD:R_0805_2012Metric, F.Cu at (77.5, 29.0)
- added R7: 4.7K, Resistor_SMD:R_0805_2012Metric, F.Cu at (78.5, 34.4)
- added R8: 10K, Resistor_SMD:R_0805_2012Metric, F.Cu at (66.3, 42.6)
- added U4: ~, Package_LGA:Bosch_LGA-8_2x2.5mm_P0.65mm_ClockwisePinNumbering, F.Cu at (74.3, 32.5)
- C2, C4: value 1µF -> 10µF; footprint Capacitor_SMD:C_1206_3216Metric -> Capacitor_SMD:C_0805_2012Metric
- C6: footprint Capacitor_SMD:C_1206_3216Metric -> Capacitor_SMD:C_0805_2012Metric
- C8, R2, R3: moved to F.Cu
- J1: value Conn_01x06_Pin -> SS445P; footprint Connector_JST:JST_SH_BM06B-SRSS-TB_1x06-1MP_P1.00mm_Vertical -> Connector_Hirose:Hirose_DF13C_CL535-0403-5-51_1x03-1MP_P1.25mm_Vertical
- J3: footprint Connector_PinHeader_2.54mm:PinHeader_1x02_P2.54mm_Vertical -> Connector_Hirose:Hirose_DF13C_CL535-0402-2-51_1x02-1MP_P1.25mm_Vertical
- J7: value Conn_01x04_Pin -> I2C BUS1; footprint Connector_PinHeader_2.54mm:PinHeader_1x04_P2.54mm_Vertical -> Connector_JST:JST_PH_S4B-PH-SM4-TB_1x04-1MP_P2.00mm_Horizontal
- J8: footprint Connector_Molex:Molex_KK-254_AE-6410-03A_1x03_P2.54mm_Vertical -> Connector_Hirose:Hirose_DF13C_CL535-0403-5-51_1x03-1MP_P1.25mm_Vertical
- moved J1 50.8 mm to (57.2, 46.3)
- moved J3 40.6 mm to (95.0, 59.5), turned to 180 degrees
- moved J7 20.4 mm to (58.4, 31.0), turned to 180 degrees
- moved C5 15.1 mm to (58.8, 53.8), turned to 90 degrees
- moved U2 14.6 mm to (65.5, 56.5), turned to -90 degrees
- moved C4 14.6 mm to (54.8, 53.8), turned to 90 degrees
- moved C2 14.3 mm to (57.0, 59.5), turned to 90 degrees
- moved C1 12.8 mm to (73.8, 59.2)
- moved R1 12.8 mm to (73.8, 53.3)
- moved U1 12.8 mm to (80.9, 53.1)
- moved J4 12.6 mm to (50.1, 55.0)
- moved Q1 11.8 mm to (82.5, 60.5)
- moved R2 11.4 mm to (87.0, 55.4)
- moved H1 11.0 mm to (49.0, 28.5)
- moved H2 11.0 mm to (49.0, 63.0)
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Connections:
- C9 pad 1: GPIO5 -> GPIO4
- J1 pad 1: GPIO4 -> +3V3
- J1 pad 2: GPIO3 -> GPIO14
- J1 pad 3: GPIO2 -> OUT-
- J7 pad 1: +3V3 -> SDA
- J7 pad 2: SDA -> SCL
- J7 pad 3: OUT- -> +3V3
- J7 pad 4: SCL -> OUT-
- R4 pad 1: GPIO5 -> GPIO4
- R5 pad 2: GPIO5 -> GPIO4
- U3 pad 12: GPIO5 -> unconnected-(U3-IO5-Pad12)
- U3 pad 14: GPIO3 -> unconnected-(U3-IO3-Pad14)
- U3 pad 15: GPIO2 -> SCL_2
- U3 pad 16: GPIO1 -> SDA_2
- U3 pad 5: GPIO13 -> unconnected-(U3-IO13-Pad5)
- U3 pad 6: unconnected-(U3-IO14-Pad6) -> GPIO14
Routing:
- net +3V3: track 149.4 -> 191.1 mm, vias 1 -> 0
- net GPIO14: track 0.00 -> 30.3 mm
- net GPIO13: track 29.0 -> 0.00 mm
- net GPIO5: track 12.1 -> 0.00 mm
- net BATT+: track 52.3 -> 62.2 mm
- net BATT-: track 46.9 -> 56.2 mm
- net GPIO3: track 8.91 -> 0.00 mm
- net SDA_2: track 0.00 -> 8.24 mm
- net SCL_2: track 0.00 -> 8.22 mm
- net SCL: track 24.5 -> 31.4 mm
- net GPIO2: track 6.65 -> 0.00 mm
- net GPIO1: track 6.01 -> 0.00 mm
- net Net-(Q1-G2): track 13.5 -> 19.4 mm
- net OUT-: track 0.00 -> 5.30 mm, vias 29 -> 49
- net SDA: track 26.7 -> 31.1 mm
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Other:
- board size 54 x 39.5 mm -> 69 x 40.5 mm
- board text added: "0.1µF"
- board text added: "100KΩ"
- board text added: "100Ω"
- board text added: "10KΩ"
- board text added: "10µF"
- board text added: "1KΩ"
- board text added: "1µF"
- board text added: "AS5600 & VEML7700"
- board text added: "Anemometer"
- board text added: "CAELUM - v2.0"
- board text added: "CAELUM - v2.0 Author: Fabiancrg"
- board text added: "DPS310"
- board text added: "DS18B20"
- board text added: "IO14"
- board text added: "Rain pulse"
- board text added: "SHT4x"
- board text removed: "1"
- board text removed: "2"
- board text removed: "3"
- board text removed: "4"
- board text removed: "CAELUM - v1.1"
- board text removed: "GPIO12"
- board text removed: "GPIO13"
- board text removed: "GPIO24"
- board text removed: "GPIOs"
- board text removed: "Pulse"
- board text removed: "VCC"
